File: lightbox-pcb.kicad_pcb (KiCad board)
At the start: 2 copper layers, 49 parts, among them J1 LED Strip, J2 LED Strip, J3 LED Strip, J4 LED Strip, J5 Control, J6 SPI_INPUT_HEADER, J7 Ant, J8 Power, Q1 BS170, Q10 BS170, Q11 BS170, Q12 BS170, Q2 BS170, Q3 BS170, Q4 BS170, Q5 BS170, Q6 BS170, Q7 BS170, Q8 BS170, Q9 BS170, SW1 SW_Slide_DPDT, SW2 SW_Slide_DPDT, U1 TLC59711, U2 ITSY_BITSY_32U4

Commit message: WILL DOES NOT LIKE SWITCH
Parts:
- added H1: MountingHole, MountingHole:MountingHole_4.3mm_M4, F.Cu at (198.6, 122.4)
- added H2: MountingHole, MountingHole:MountingHole_4.3mm_M4, F.Cu at (117.6, 122.4)
- added H3: MountingHole, MountingHole:MountingHole_4.3mm_M4, F.Cu at (198.6, 80.8)
- added H4: MountingHole, MountingHole:MountingHole_4.3mm_M4, F.Cu at (117.6, 80.8)
- J1, J2, J3, J4: footprint Connector_PinHeader_2.54mm:PinHeader_1x03_P2.54mm_Vertical -> Connector_Phoenix_MC:PhoenixContact_MC_1,5_4-G-3.5_1x04_P3.50mm_Horizontal
- Q1, Q10, Q11, Q12, Q2, Q3, Q4, Q5, Q6, Q7, Q8, Q9: value BS170 -> DMN13H750S; footprint Package_TO_SOT_THT:TO-92_HandSolder -> Package_TO_SOT_SMD:SOT-23
- R1, R10, R11, R12, R13, R14, R15, R16, R17, R18, R19, R2, R20, R21, R22, R23, R24, R26, R3, R4, R5, R6, R7, R8, R9: footprint will:Dan_Through_Hole_Res -> Resistor_SMD:R_0805_2012Metric_Pad1.20x1.40mm_HandSolder
- SW1, SW2: moved to B.Cu
- moved J8 103.1 mm to (118.1, 98.6)
- moved R12 99.5 mm to (170.8, 88.5)
- moved R9 95.2 mm to (174.6, 88.5)
- moved R10 93.2 mm to (177.2, 88.5)
- moved R11 91.5 mm to (160.8, 66.3)
- moved J2 91.1 mm to (172.9, 81.0), turned to 180 degrees
- moved R7 88.3 mm to (180.3, 88.5)
- moved Q5 88.1 mm to (173.7, 66.6)
- moved Q6 87.8 mm to (159.9, 62.2)
- moved R8 86.7 mm to (182.9, 88.5)
- moved Q4 81.0 mm to (179.1, 66.3)
- moved R26 71.4 mm to (191.8, 113.9), turned to -90 degrees
- moved U2 71.2 mm to (184.8, 101.6)
- moved J5 66.5 mm to (189.5, 78.1)
- moved J7 60.2 mm to (201.5, 78.8)
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Connections:
- Q1 pad 1: Net-(J1-B) -> Net-(Q1-G)
- Q1 pad 2: Net-(Q1-G) -> GND
- Q1 pad 3: GND -> Net-(J1-B)
- Q10 pad 1: Net-(J4-B) -> Net-(Q10-G)
- Q10 pad 2: Net-(Q10-G) -> GND
- Q10 pad 3: GND -> Net-(J4-B)
- Q11 pad 1: Net-(J4-G) -> Net-(Q11-G)
- Q11 pad 2: Net-(Q11-G) -> GND
- Q11 pad 3: GND -> Net-(J4-G)
- Q12 pad 1: Net-(J4-R) -> Net-(Q12-G)
- Q12 pad 2: Net-(Q12-G) -> GND
- Q12 pad 3: GND -> Net-(J4-R)
- Q2 pad 1: Net-(J1-G) -> Net-(Q2-G)
- Q2 pad 2: Net-(Q2-G) -> GND
- Q2 pad 3: GND -> Net-(J1-G)
- Q3 pad 1: Net-(J1-R) -> Net-(Q3-G)
- Q3 pad 2: Net-(Q3-G) -> GND
- Q3 pad 3: GND -> Net-(J1-R)
- Q4 pad 1: Net-(J2-B) -> Net-(Q4-G)
- Q4 pad 2: Net-(Q4-G) -> GND
- Q4 pad 3: GND -> Net-(J2-B)
- Q5 pad 1: Net-(J2-G) -> Net-(Q5-G)
- Q5 pad 2: Net-(Q5-G) -> GND
- Q5 pad 3: GND -> Net-(J2-G)
- Q6 pad 1: Net-(J2-R) -> Net-(Q6-G)
- Q6 pad 2: Net-(Q6-G) -> GND
- Q6 pad 3: GND -> Net-(J2-R)
- Q7 pad 1: Net-(J3-B) -> Net-(Q7-G)
- Q7 pad 2: Net-(Q7-G) -> GND
- Q7 pad 3: GND -> Net-(J3-B)
- Q8 pad 1: Net-(J3-G) -> Net-(Q8-G)
- Q8 pad 2: Net-(Q8-G) -> GND
- Q8 pad 3: GND -> Net-(J3-G)
- Q9 pad 1: Net-(J3-R) -> Net-(Q9-G)
- Q9 pad 2: Net-(Q9-G) -> GND
- Q9 pad 3: GND -> Net-(J3-R)
Routing:
- net /SR1: track 121.1 -> 0.00 mm
- net /SG1: track 105.2 -> 0.00 mm
- net /SB1: track 88.3 -> 0.00 mm
- net /SR0: track 69.9 -> 0.00 mm
- net /SG0: track 63.3 -> 0.00 mm
- net /SB0: track 56.7 -> 0.00 mm
- net Net-(U1-V+): track 0.00 -> 24.3 mm
- net +5V: track 0.00 -> 23.2 mm
- net Net-(J5-Speed): track 0.00 -> 19.0 mm
- net Net-(J5-Bright): track 0.00 -> 17.3 mm
- net Net-(J1-B): track 15.3 -> 0.00 mm
- net Net-(J1-R): track 15.0 -> 0.00 mm
- net +12V: track 0.00 -> 13.3 mm
- net Net-(Q3-G): track 12.8 -> 0.00 mm
- net Net-(Q1-G): track 14.7 -> 3.45 mm
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- added copper zone on F.Cu, net +12V
- added copper zone on B.Cu, net GND
Other:
- board outline added: 90.2 x 50.8 mm
- board text added: "WILL DOES NOT LIKE SWITCH"
