File: lightbox-pcb.kicad_sch (KiCad schematic)
At the start: 58 parts, among them J1 0, J10 Control, J11 Power, J12 Extern, J13 LED Strip, J14 LED Strip, J15 LED Strip, J16 Ant, J2 LED Strip, J3 1, J4 3, J5 2, J9 Control, Q1 BS170, Q10 BS170, Q11 BS170, Q12 BS170, Q2 BS170, Q3 BS170, Q4 BS170, Q5 BS170, Q6 BS170, Q7 BS170, Q8 BS170, Q9 BS170

Commit message: wrong files
Parts:
- removed J1: 0, symbol Connector:Conn_01x03_Socket
- removed J12: Extern, symbol Connector:Conn_01x05_Pin
- removed J3: 1, symbol Connector:Conn_01x03_Socket
- removed J4: 3, symbol Connector:Conn_01x03_Socket
- removed J5: 2, symbol Connector:Conn_01x03_Socket
- removed J6: ~, symbol Connector:Conn_01x05_Socket
- removed J7, J8: ~, symbol Connector:Conn_01x14_Socket
- removed SW1, SW3: ~, symbol Switch:SW_DPST_x2
- added J6: SPI_INPUT_HEADER, Connector_PinHeader_2.54mm:PinHeader_1x04_P2.54mm_Vertical, symbol Connector:Conn_01x04_Pin
- added SW1, SW2: SW_Slide_DPDT, Button_Switch_THT:SW_CK_JS202011CQN_DPDT_Straight, symbol Switch:SW_Slide_DPDT
- added U1: TLC59711, will:TLC59711, symbol 4015:TLC59711
- added U2: ITSY_BITSY_32U4, will:Itsy_bitsy_32u4, symbol 4015:Itsy_bitsy_32u4
- J1: renamed from J2; footprint (none) -> Connector_PinHeader_2.54mm:PinHeader_1x03_P2.54mm_Vertical
- J2: renamed from J13; footprint (none) -> Connector_PinHeader_2.54mm:PinHeader_1x03_P2.54mm_Vertical
- J3: renamed from J14; footprint (none) -> Connector_PinHeader_2.54mm:PinHeader_1x03_P2.54mm_Vertical
- J4: renamed from J15; footprint (none) -> Connector_PinHeader_2.54mm:PinHeader_1x03_P2.54mm_Vertical
- J5: renamed from J9; footprint (none) -> Connector_PinHeader_2.54mm:PinHeader_1x04_P2.54mm_Vertical
- J7: renamed from J16; footprint (none) -> Connector_PinHeader_2.54mm:PinHeader_1x01_P2.54mm_Vertical
- J8: renamed from J11; footprint (none) -> Connector_Samtec_HPM_THT:Samtec_HPM-02-01-x-S_Straight_1x02_Pitch5.08mm
- J9: renamed from J10; footprint (none) -> Connector_Phoenix_MSTB:PhoenixContact_MSTBVA_2,5_4-G-5,08_1x04_P5.08mm_Vertical
- Q1: renamed from Q3; footprint Package_TO_SOT_THT:TO-92_Inline -> Package_TO_SOT_THT:TO-92_HandSolder
- Q10, Q11, Q12, Q2, Q4, Q5, Q6, Q7, Q8, Q9: footprint Package_TO_SOT_THT:TO-92_Inline -> Package_TO_SOT_THT:TO-92_HandSolder
- Q3: renamed from Q1; footprint Package_TO_SOT_THT:TO-92_Inline -> Package_TO_SOT_THT:TO-92_HandSolder
- R1: renamed from R3; footprint (none) -> will:Dan_Through_Hole_Res
- R10: renamed from R12; footprint (none) -> will:Dan_Through_Hole_Res
- R11: renamed from R13; footprint (none) -> will:Dan_Through_Hole_Res
- R12: renamed from R14; footprint (none) -> will:Dan_Through_Hole_Res
- R13: renamed from R15; footprint (none) -> will:Dan_Through_Hole_Res
- R14: renamed from R16; footprint (none) -> will:Dan_Through_Hole_Res
- R15: renamed from R17; footprint (none) -> will:Dan_Through_Hole_Res
- R16: renamed from R18; footprint (none) -> will:Dan_Through_Hole_Res
- R17: renamed from R19; footprint (none) -> will:Dan_Through_Hole_Res
- R18: renamed from R20; footprint (none) -> will:Dan_Through_Hole_Res
- R19: renamed from R21; footprint (none) -> will:Dan_Through_Hole_Res
- R2: renamed from R6; footprint (none) -> will:Dan_Through_Hole_Res
- R20: renamed from R22; footprint (none) -> will:Dan_Through_Hole_Res
- R21: renamed from R23; footprint (none) -> will:Dan_Through_Hole_Res
- R22: renamed from R24; footprint (none) -> will:Dan_Through_Hole_Res
- R23: renamed from R25; footprint (none) -> will:Dan_Through_Hole_Res
- R24: renamed from R26; footprint (none) -> will:Dan_Through_Hole_Res
- R25: renamed from R8; footprint (none) -> will:Dan_Through_Hole_Res
- R26: renamed from R7; footprint (none) -> will:Dan_Through_Hole_Res
- R3: renamed from R2; footprint (none) -> will:Dan_Through_Hole_Res
- R4: renamed from R5; footprint (none) -> will:Dan_Through_Hole_Res
- R5: renamed from R1; footprint (none) -> will:Dan_Through_Hole_Res
- R6: renamed from R4; footprint (none) -> will:Dan_Through_Hole_Res
- R7: renamed from R9; footprint (none) -> will:Dan_Through_Hole_Res
- R8: renamed from R10; footprint (none) -> will:Dan_Through_Hole_Res
- R9: renamed from R11; footprint (none) -> will:Dan_Through_Hole_Res
- renumbered RV2 to RV1, RV1 to RV2
Connections:
- net +12V: now also U2.28 (BAT)
- net +5V: now also SW1.1 (A), U2.2 (5V)
- net EN: now also U2.24 (12)
- net GND: now also J6.4 (Gnd), U1.1 (GND), U2.27 (G), U2.4 (GND)
- net MOSI: now also SW2.1 (A), U2.12 (MOSI)
- net SB0: now also U1.10 (B0)
- net SB1: now also U1.13 (B1)
- net SB2: now also U1.16 (B2)
- net SB3: now also U1.19 (B3)
- net SCK: now also SW2.6 (C), U2.11 (SCK)
- net SG0: now also U1.9 (G0)
- net SG1: now also U1.12 (G1)
- net SG2: now also U1.15 (G2)
- net SG3: now also U1.18 (G3)
- net SR0: now also U1.8 (R0)
- net SR1: now also U1.11 (R1)
- net SR2: now also U1.14 (R2)
- net SR3: now also U1.17 (R3)
- net at J5.3 (Bright): now also U2.7 (Pin_7)
- net at J5.4 (Speed): now also U2.9 (A4)
- net at J7.1 (Pin_1): now also U2.5 (A0)
- new net: SW1.2 (B), U1.2 (VCC), U1.3 (V+)
- new net: SW2.5 (B), U1.4 (CI)
- new net: SW2.2 (B), U1.5 (DI)
- new net: J6.1 (DI), SW2.3 (C)
- new net: J6.2 (CI), SW2.4 (A)
- new net: J6.3 (Vcc), SW1.3 (C)
Other:
- note added: "PinHeader Parts In library are the best to use for generic 2.54mm headers"
- note removed: "Itsy Bitsy 32u4 5V Adafruit 3677"
- note removed: "Note header"
- note removed: "TLC59711 Breakout Adafruit 1455"
- title: (none) -> Dan lightbox driver board
- moved on the sheet: J1, J2, J3, J4, J5, J7, J8, J9, R26

Commit message: WILL DOES NOT LIKE SWITCH
Parts:
- added H1, H2, H3, H4: MountingHole, MountingHole:MountingHole_4.3mm_M4, symbol Mechanical:MountingHole
- J1, J2, J3, J4: footprint Connector_PinHeader_2.54mm:PinHeader_1x03_P2.54mm_Vertical -> Connector_Phoenix_MC:PhoenixContact_MC_1,5_4-G-3.5_1x04_P3.50mm_Horizontal
- Q1, Q10, Q11, Q12, Q2, Q3, Q4, Q5, Q6, Q7, Q8, Q9: value BS170 -> DMN13H750S; footprint Package_TO_SOT_THT:TO-92_HandSolder -> Package_TO_SOT_SMD:SOT-23; symbol Transistor_FET:BS170 -> Transistor_FET:DMN13H750S
- R1, R10, R11, R12, R13, R14, R15, R16, R17, R18, R19, R2, R20, R21, R22, R23, R24, R26, R3, R4, R5, R6, R7, R8, R9: footprint will:Dan_Through_Hole_Res -> Resistor_SMD:R_0805_2012Metric_Pad1.20x1.40mm_HandSolder
Connections:
- net GND: now also Q1.2 (S), Q10.2 (S), Q11.2 (S), Q12.2 (S), Q2.2 (S), Q3.2 (S), Q4.2 (S), Q5.2 (S), Q6.2 (S), Q7.2 (S), Q8.2 (S), Q9.2 (S); no longer Q1.3 (S), Q10.3 (S), Q11.3 (S), Q12.3 (S), Q2.3 (S), Q3.3 (S), Q4.3 (S), Q5.3 (S), Q6.3 (S), Q7.3 (S), Q8.3 (S), Q9.3 (S)
- net at R10.1, R9.1: now also Q5.1 (G); no longer Q5.2 (G)
- net at R3.1, R4.1: now also Q2.1 (G); no longer Q2.2 (G)
- net at J1.2 (G): now also Q2.3 (D); no longer Q2.1 (D)
- net at R23.1, R24.1: now also Q12.1 (G); no longer Q12.2 (G)
- net at R17.1, R18.1: now also Q9.1 (G); no longer Q9.2 (G)
- net at Q1.1 (G): now also R1.1, R2.1; no longer J1.3 (B)
- net at R19.1, R20.1: now also Q10.1 (G); no longer Q10.2 (G)
- net at R21.1, R22.1: now also Q11.1 (G); no longer Q11.2 (G)
- net at R7.1, R8.1: now also Q4.1 (G); no longer Q4.2 (G)
- net at R15.1, R16.1: now also Q8.1 (G); no longer Q8.2 (G)
- net at J3.2 (G): now also Q8.3 (D); no longer Q8.1 (D)
- net at J4.1 (R): now also Q12.3 (D); no longer Q12.1 (D)
- net at R13.1, R14.1: now also Q7.1 (G); no longer Q7.2 (G)
- net at R5.1, R6.1: now also Q3.1 (G); no longer Q3.2 (G)
- net at J2.1 (R): now also Q6.3 (D); no longer Q6.1 (D)
- net at J2.2 (G): now also Q5.3 (D); no longer Q5.1 (D)
- net at J2.3 (B): now also Q4.3 (D); no longer Q4.1 (D)
- net at R11.1, R12.1: now also Q6.1 (G); no longer Q6.2 (G)
- net at J4.2 (G): now also Q11.3 (D); no longer Q11.1 (D)
- net at J4.3 (B): now also Q10.3 (D); no longer Q10.1 (D)
- net at J1.1 (R): now also Q3.3 (D); no longer Q3.1 (D)
- net at J3.1 (R): now also Q9.3 (D); no longer Q9.1 (D)
- net at J3.3 (B): now also Q7.3 (D); no longer Q7.1 (D)
- new net: J1.3 (B), Q1.3 (D)
